File: Metro M7 RT1011 SD rev A.kicad_pcb (KiCad board)
At the start: 2 copper layers, 68.6 x 53.3 mm, 101 parts, among them IC2 IMX_RT1010, IC4 RESET_SUPERVISORAPX80X_SA, J2 Conn_ARM_JTAG_SWD_10, SW1 SPDT_RA, SW2 DIP2, T2 DMP3098L-7, U1 NCP1117ST50T3G, U2 LP2985-XXDBVR, U3 W25Q64JV, X1 MICROSD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

Commit message: v2
Other:
- board text added: "ckd.tech/1011-trace/v2"
- board text removed: "ckd.tech/1011-trace/v1"
Changed lines of the file:
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@@
     (fp_line (start 3.6 2) (end -7.3 2)
       (stroke (width 0.2032) (type solid)) (layer "F.Fab"))
-    (pad "GND" thru_hole oval (at -2.9 -2.54 270) (size 5.4 2.7) (drill 0.9) (layers "*.Cu" "*.Mask")
+    (pad "GND" thru_hole oval (at -2.9 -2.54 270) (size 5.4 2.7) (drill oval 3.5 1) (layers "*.Cu" "*.Mask")
       (net 2 "GND") (pinfunction "GND") (pintype "power_in") (solder_mask_margin 0.0508) (thermal_bridge_angle 45))
-    (pad "GNDBREAK" thru_hole oval (at 0 2.16) (size 5.4 2.7) (drill 0.9) (layers "*.Cu" "*.Mask")
+    (pad "GNDBREAK" thru_hole oval (at 0 2.16) (size 5.4 2.7) (drill oval 3.5 1) (layers "*.Cu" "*.Mask")
       (net 2 "GND") (pinfunction "GNDBREAK") (pintype "power_in") (solder_mask_margin 0.0508) (thermal_bridge_angle 45))
-    (pad "PWR" thru_hole oval (at 3 -2.54 270) (size 5.4 2.7) (drill 0.9) (layers "*.Cu" "*.Mask")
+    (pad "PWR" thru_hole oval (at 3 -2.54 270) (size 5.4 2.7) (drill oval 3.5 1) (layers "*.Cu" "*.Mask")
       (net 21 "Net-(D1-PadA)") (pinfunction "PWR") (pintype "power_in") (solder_mask_margin 0.0508) (thermal_bridge_angle 45))
   )
@@
     (property "Sheetfile" "Metro M7 RT1011 SD rev A.kicad_sch")
     (property "Sheetname" "Metro M7 RT1011 SD rev A_0")
+    (attr exclude_from_pos_files exclude_from_bom)
     (fp_text reference "LED1" (at -1.905 -2.159) (layer "F.SilkS") hide
         (effects (font (size 0.896031 0.896031) (thickness 0.119969)) (justify right))
@@
     (pad "B8" smd rect (at -1.75 -2.275 270) (size 0.275 1.15) (layers "F.Cu" "F.Paste" "F.Mask")
       (net 86 "unconnected-(X4-SBU2-PadB8)") (pinfunction "SBU2") (pintype "bidirectional+no_connect") (solder_mask_margin 0.0508) (thermal_bridge_angle 45))
-    (pad "M1" thru_hole oval (at -4.32 -1.7) (size 2 1) (drill 0.6) (layers "*.Cu" "*.Mask")
+    (pad "M1" thru_hole oval (at -4.32 -1.7) (size 2 1) (drill oval 1.7 0.6) (layers "*.Cu" "*.Mask")
       (solder_mask_margin 0.0508) (thermal_bridge_angle 45))
-    (pad "M2" thru_hole oval (at 4.32 -1.7) (size 2 1) (drill 0.6) (layers "*.Cu" "*.Mask")
+    (pad "M2" thru_hole oval (at 4.32 -1.7) (size 2 1) (drill oval 1.7 0.6) (layers "*.Cu" "*.Mask")
       (solder_mask_margin 0.0508) (thermal_bridge_angle 45))
-    (pad "M3" thru_hole oval (at -4.32 2.48) (size 2 1) (drill 0.6) (layers "*.Cu" "*.Mask")
+    (pad "M3" thru_hole oval (at -4.32 2.48) (size 2 1) (drill oval 1.7 0.6) (layers "*.Cu" "*.Mask")
       (solder_mask_margin 0.0508) (thermal_bridge_angle 45))
-    (pad "M4" thru_hole oval (at 4.32 2.48) (size 2 1) (drill 0.6) (layers "*.Cu" "*.Mask")
+    (pad "M4" thru_hole oval (at 4.32 2.48) (size 2 1) (drill oval 1.7 0.6) (layers "*.Cu" "*.Mask")
       (solder_mask_margin 0.0508) (thermal_bridge_angle 45))
   )
@@
     (effects (font (size 0.8 0.8) (thickness 0.15)) (justify right))
   )
-  (gr_text "ckd.tech/1011-trace/v1" (at 118.1481 100.6856) (layer "F.SilkS")
+  (gr_text "ckd.tech/1011-trace/v2" (at 118.1481 100.6856) (layer "F.SilkS")
     (effects (font (size 1 1) (thickness 0.1)) (justify left bottom))
   )
