File: Metro M7 RT1011 SD rev A.kicad_sch (KiCad schematic)
At the start: 94 parts, among them IC2 IMX_RT1010, IC4 RESET_SUPERVISORAPX80X_SA, J2 Conn_ARM_JTAG_SWD_10, SW1 SPDT_RA, SW2 DIP2, T2 DMP3098L-7, U1 NCP1117ST50T3G, U2 LP2985-XXDBVR, U3 W25Q64JV, X1 MICROSD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

Commit message: v2
Parts:
- added C1: 0.1uF, Metro M7 RT1011 SD rev A:0603-NO, symbol Metro M7 RT1011 SD rev A-eagle-import:CAP_CERAMIC0603_NO
Connections:
- net GND: now also C1.1
- net at J2.11 (VTpwr): now also J2.13 (VTpwr), C1.2
- no-connect marks 25 -> 23
Other:
- note added: "Decouple to allow signal (AC) return path."
Changed lines of the file:
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@@
   (junction (at 233.68 45.72) (diameter 0) (color 0 0 0 0)
   )
+  (junction (at 354.33 196.85) (diameter 0) (color 0 0 0 0)
+  )
   (junction (at 111.76 78.74) (diameter 0) (color 0 0 0 0)
   )
@@
   (no_connect (at 68.58 187.96))
   (no_connect (at 58.42 144.78))
-  (no_connect (at 351.79 199.39))
-  (no_connect (at 354.33 199.39))
   (no_connect (at 190.5 233.68))
   (no_connect (at 190.5 254))
@@
     (stroke (width 0) (type default))
   )
+  (wire (pts (xy 351.79 199.39) (xy 351.79 196.85))
+    (stroke (width 0) (type default))
+  )
   (wire (pts (xy 190.5 248.92) (xy 223.52 248.92))
     (stroke (width 0.1524) (type solid))
@@
     (stroke (width 0.1524) (type solid))
   )
+  (wire (pts (xy 354.33 196.85) (xy 354.33 199.39))
+    (stroke (width 0) (type default))
+  )
   (wire (pts (xy 215.9 256.54) (xy 190.5 256.54))
     (stroke (width 0.1524) (type solid))
@@
     (stroke (width 0.1524) (type solid))
   )
+  (wire (pts (xy 354.33 195.58) (xy 354.33 196.85))
+    (stroke (width 0) (type default))
+  )
   (wire (pts (xy 218.44 254) (xy 218.44 261.62))
     (stroke (width 0.1524) (type solid))
@@
     (stroke (width 0.1524) (type solid))
   )
+  (wire (pts (xy 351.79 196.85) (xy 354.33 196.85))
+    (stroke (width 0) (type default))
+  )
   (wire (pts (xy 119.38 238.76) (xy 124.46 238.76))
     (stroke (width 0.1524) (type solid))
@@
     (effects (font (size 1.778 1.5113)) (justify left))
   )
+  (text "Decouple to allow signal (AC)\nreturn path." (at 358.14 191.77 0)
+    (effects (font (size 1.27 1.27)) (justify left bottom))
+  )
   (text "3" (at 241.3 261.62 0)
     (effects (font (size 1.778 1.5113)) (justify left))
@@
   )
   (text "X" (at 68.58 187.96 0)
-    (effects (font (size 1.778 1.5113)) (justify right))
+    (effects (font (size 1.778 1.5113)) (justify right bottom))
   )
   (text "Limor Fried & Dean M." (at 350.52 259.08 0)
@@
     )
   )
+  (symbol (lib_id "Metro M7 RT1011 SD rev A-eagle-import:GND") (at 354.33 185.42 180) (unit 1)
+    (in_bom yes) (on_board yes) (dnp no) (fields_autoplaced)
+    (property "Reference" "#GND018" (at 354.33 185.42 0)
+      (effects (font (size 1.27 1.27)) hide)
+    )
+    (property "Value" "GND" (at 354.33 182.88 0)
+      (effects (font (size 1.778 1.5113)))
+    )
+    (property "Footprint" "" (at 354.33 185.42 0)
+      (effects (font (size 1.27 1.27)) hide)
+    )
+    (property "Datasheet" "" (at 354.33 185.42 0)
+      (effects (font (size 1.27 1.27)) hide)
+    )
+    (pin "1")
+    (instances
+      (project "Metro M7 RT1011 SD rev A"
+        (path "/ade93230-af5f-4a46-9a5f-971407796e9c"
+          (reference "#GND018") (unit 1)
+        )
+      )
+    )
+  )
   (symbol (lib_id "Metro M7 RT1011 SD rev A-eagle-import:CAP_CERAMIC0805-NOOUTLINE") (at 134.62 198.12 0) (unit 1)
     (in_bom yes) (on_board yes) (dnp no)
@@
     )
   )
+  (symbol (lib_id "Metro M7 RT1011 SD rev A-eagle-import:CAP_CERAMIC0603_NO") (at 354.33 193.04 0) (unit 1)
+    (in_bom yes) (on_board yes) (dnp no)
+    (property "Reference" "C1" (at 352.04 191.79 90)
+      (effects (font (size 1.27 1.27)))
+    )
+    (property "Value" "0.1uF" (at 356.63 191.79 90)
+      (effects (font (size 1.27 1.27)))
+    )
+    (property "Footprint" "Metro M7 RT1011 SD rev A:0603-NO" (at 354.33 193.04 0)
+      (effects (font (size 1.27 1.27)) hide)
+    )
+    (property "Datasheet" "" (at 354.33 193.04 0)
+      (effects (font (size 1.27 1.27)) hide)
+    )
+    (pin "1")
+    (pin "2")
+    (instances
+      (project "Metro M7 RT1011 SD rev A"
+        (path "/ade93230-af5f-4a46-9a5f-971407796e9c"
+          (reference "C1") (unit 1)
+        )
+      )
+    )
+  )
   (symbol (lib_id "Metro M7 RT1011 SD rev A-eagle-import:CAP_CERAMIC0603_NO") (at 137.16 241.3 0) (unit 1)
     (in_bom yes) (on_board yes) (dnp no)
@@
     (pin "11")
     (pin "12")
+    (pin "13")
     (pin "14")
     (pin "15")
@@
     (pin "2")
     (pin "20")
-    (pin "13")
     (pin "3")
     (pin "4")
